Commit message: first fix of the sim physics with the casters

File: hamr_description/urdf/hamr_gazebo.xacro (robot description, xacro)
@@ -2,30 +2,33 @@
 <robot name="hamr" xmlns:xacro="http://www.ros.org/wiki/xacro">
     <gazebo reference="right_wheel_link">
-        <mu1 value="1.0" />
-        <mu2 value="1.0" />
+        <mu1 value="0.9" />
+        <mu2 value="0.9" />
     </gazebo>
     <gazebo reference="left_wheel_link">
-        <mu1 value="1.0" />
-        <mu2 value="1.0" />
+        <mu1 value="0.9" />
+        <mu2 value="0.9" />
     </gazebo>
     <gazebo reference="right_caster_link">
-        <mu1 value="0.2" />
-        <mu2 value="0.2" />
+        <mu1 value="0.000002" />
+        <mu2 value="0.02" />
     </gazebo>
     <gazebo reference="left_caster_link">
-        <mu1 value="0.2" />
-        <mu2 value="0.2" />
+        <mu1 value="0.000002" />
+        <mu2 value="0.02" />
     </gazebo>
     <gazebo reference="right_caster_wheel_link">
-        <mu1 value="0.8" />
-        <mu2 value="0.8" />
+        <mu1 value="0.9"/>  <!-- lateral -->
+        <mu2 value="0.2"/>   <!-- rolling -->
+        <fdir1 value="0 0 1" />
     </gazebo>
     <gazebo reference="left_caster_wheel_link">
-        <mu1 value="0.8" />
-        <mu2 value="0.8" />
+        <mu1 value="0.9"/>  <!-- lateral -->
+        <mu2 value="0.2"/>   <!-- rolling -->
+        <fdir1 value="0 0 1" />
     </gazebo>
     <gazebo reference="turret_link">
         <mu2 value="0.6" />
         <mu1 value="0.6" />
+        <fdir1 value="0 0 1" />
     </gazebo>
     <gazebo>
@@ -90,5 +93,5 @@
         <left_joint>base_left_wheel_joint</left_joint>
         <right_joint>base_right_wheel_joint</right_joint>
-        <wheel_separation>0.308</wheel_separation>
+        <wheel_separation>0.299</wheel_separation>
         <wheel_radius>0.0762</wheel_radius>
         <frame_id>odom</frame_id>

File: hamr_description/urdf/hamr_sw.xacro (robot description, xacro)
@@ -60,5 +60,5 @@
         rpy="0 1.5707963267949 0" />
       <mass
-        value="0.201354791790072" />
+        value="${3 * 0.201354791790072}" />
       <inertia
         ixx="0.000633771005763446"
@@ -86,8 +86,9 @@
       <origin
         xyz="0 0 0"
-        rpy="0 1.5707963267949 0" />
-      <geometry>
-        <mesh
-          filename="package://hamr_description/meshes/right_wheel_link.stl" />
+        rpy="0 0 0" />
+      <geometry>
+        <!-- <mesh
+          filename="package://hamr_description/meshes/right_wheel_link.stl" /> -->
+        <cylinder radius="0.0762" length="0.0254" />
       </geometry>
     </collision>
@@ -110,5 +111,5 @@
         rpy="0 ${pi} 0" />
       <mass
-        value="0.201354790396108" />
+        value="${3 * 0.201354790396108}" />
       <inertia
         ixx="0.000327993572579979"
@@ -121,5 +122,5 @@
     <visual>
       <origin
-        xyz="0 0 0"
+        xyz="0 0 ${0.0254 / 2.0}"
         rpy="0 ${pi} 0" />
       <geometry>
@@ -138,6 +139,7 @@
         rpy="0 ${pi} 0" />
       <geometry>
-        <mesh
-          filename="package://hamr_description/meshes/left_wheel_link.stl" />
+        <!-- <mesh
+          filename="package://hamr_description/meshes/left_wheel_link.stl" /> -->
+        <cylinder radius="0.0762" length="0.0254" />
       </geometry>
     </collision>
@@ -145,5 +147,5 @@
   <joint name="base_left_wheel_joint" type="continuous">
     <origin
-      xyz="0.365456260020371 -0.0880218689795108 -0.044451036743372"
+      xyz="${0.365456260020371 - 0.0254 / 2.0} -0.0880218689795108 -0.044451036743372"
       rpy="0 1.5707963267949 0" />
     <parent
@@ -203,4 +205,6 @@
     <axis
       xyz="0 1 0" />
+    <!-- <dynamics damping="2.0" friction="0.0"/>
+    <limit effort="5.0" velocity="10.0"/> -->
   </joint>
   <link name="right_caster_wheel_link">
@@ -238,6 +242,8 @@
         rpy="0 0 0" />
       <geometry>
-        <mesh
-          filename="package://hamr_description/meshes/right_caster_wheel_link.stl" />
+        <!-- <mesh
+          filename="package://hamr_description/meshes/right_caster_wheel_link.stl" /> -->
+        <cylinder radius="0.0508" length="0.0222" />
+        <!-- <sphere radius="0.0508" /> -->
       </geometry>
     </collision>
@@ -253,4 +259,6 @@
     <axis
       xyz="0 0 1" />
+    <!-- <dynamics damping="0.2" friction="0.0"/> -->
+    <!-- <limit effort="2.0" velocity="20.0"/> -->
   </joint>
   <link name="left_caster_link">
@@ -303,4 +311,6 @@
     <axis
       xyz="0 1 0" />
+    <!-- <dynamics damping="2.0" friction="0.0"/>
+    <limit effort="5.0" velocity="10.0"/> -->
   </joint>
   <link name="left_caster_wheel_link">
@@ -338,6 +348,8 @@
         rpy="0 0 0" />
       <geometry>
-        <mesh
-          filename="package://hamr_description/meshes/left_caster_wheel_link.stl" />
+        <!-- <mesh
+          filename="package://hamr_description/meshes/left_caster_wheel_link.stl" /> -->
+        <cylinder radius="0.0508" length="0.0222" />
+        <!-- <sphere radius="0.0508" /> -->
       </geometry>
     </collision>
@@ -353,4 +365,6 @@
     <axis
       xyz="0 0 1" />
+    <!-- <dynamics damping="0.2" friction="0.0"/>
+    <limit effort="2.0" velocity="20.0"/> -->
   </joint>
   <link name="turret_link">
