Commit message: Fully fixed and tuned Penn HAMR. Works with varying angles and works in maze. Next steps: - Varying angles in A* - Smoothed traj post A*? Not always wanted tho - Implement ROS2 Actions and Services for more advanced modes and autonomy - for example find the way out of the maze, always keep the heading angle at a given angle, ...

File: hamr_description/urdf/hamr_sw.xacro (robot description, xacro)
@@ -8,5 +8,5 @@
   <joint name="base_footprint_base_joint" type="fixed">
     <origin
-      xyz="0 0 0.12064984794"
+      xyz="-0.284843388017437 -0.203598611982565 0.12064984794"
       rpy="0 0 ${pi/2.0}" />
     <parent
@@ -60,5 +60,5 @@
         rpy="0 1.5707963267949 0" />
       <mass
-        value="${10 * 0.201354791790072}" />
+        value="0.201354791790072" />
       <inertia
         ixx="0.000633771005763446"
@@ -86,9 +86,8 @@
       <origin
         xyz="0 0 0"
-        rpy="0 0 0" />
-      <geometry>
-        <!-- <mesh
-          filename="package://hamr_description/meshes/right_wheel_link.stl" /> -->
-        <cylinder radius="0.0762" length="0.0254" />
+        rpy="0 1.5707963267949 0" />
+      <geometry>
+        <mesh
+          filename="package://hamr_description/meshes/right_wheel_link.stl" />
       </geometry>
     </collision>
@@ -111,5 +110,5 @@
         rpy="0 ${pi} 0" />
       <mass
-        value="${10 * 0.201354790396108}" />
+        value="0.201354790396108" />
       <inertia
         ixx="0.000327993572579979"
@@ -139,7 +138,6 @@
         rpy="0 ${pi} 0" />
       <geometry>
-        <!-- <mesh
-          filename="package://hamr_description/meshes/left_wheel_link.stl" /> -->
-        <cylinder radius="0.0762" length="0.0254" />
+        <mesh
+          filename="package://hamr_description/meshes/left_wheel_link.stl" />
       </geometry>
     </collision>
@@ -205,6 +203,4 @@
     <axis
       xyz="0 1 0" />
-    <!-- <dynamics damping="2.0" friction="0.0"/>
-    <limit effort="5.0" velocity="10.0"/> -->
   </joint>
   <link name="right_caster_wheel_link">
@@ -242,8 +238,6 @@
         rpy="0 0 0" />
       <geometry>
-        <!-- <mesh
-          filename="package://hamr_description/meshes/right_caster_wheel_link.stl" /> -->
-        <cylinder radius="0.0508" length="0.0222" />
-        <!-- <sphere radius="0.0508" /> -->
+        <mesh
+          filename="package://hamr_description/meshes/right_caster_wheel_link.stl" />
       </geometry>
     </collision>
@@ -259,6 +253,4 @@
     <axis
       xyz="0 0 1" />
-    <!-- <dynamics damping="0.2" friction="0.0"/> -->
-    <!-- <limit effort="2.0" velocity="20.0"/> -->
   </joint>
   <link name="left_caster_link">
@@ -311,6 +303,4 @@
     <axis
       xyz="0 1 0" />
-    <!-- <dynamics damping="2.0" friction="0.0"/>
-    <limit effort="5.0" velocity="10.0"/> -->
   </joint>
   <link name="left_caster_wheel_link">
@@ -348,8 +338,6 @@
         rpy="0 0 0" />
       <geometry>
-        <!-- <mesh
-          filename="package://hamr_description/meshes/left_caster_wheel_link.stl" /> -->
-        <cylinder radius="0.0508" length="0.0222" />
-        <!-- <sphere radius="0.0508" /> -->
+        <mesh
+          filename="package://hamr_description/meshes/left_caster_wheel_link.stl" />
       </geometry>
     </collision>
@@ -365,6 +353,4 @@
     <axis
       xyz="0 0 1" />
-    <!-- <dynamics damping="0.2" friction="0.0"/>
-    <limit effort="2.0" velocity="20.0"/> -->
   </joint>
   <link name="turret_link">

Commit message: Added Custom Map generation in Gazebo from grayscale heightmap. Also edited urdf to simplify geometric shapes to be able to run sim. Other minor changes in the python controller, added more points in PRM and updated README with the added export command for maps.

File: hamr_description/urdf/hamr_sw.xacro (robot description, xacro)
@@ -46,9 +46,10 @@
     <collision>
       <origin
-        xyz="0 0 0"
-        rpy="0 0 0" />
-      <geometry>
-        <mesh
-          filename="package://hamr_description/meshes/base_link.stl" />
+        xyz="0.198549611345678 -0.271316507443243 0.0289830936800706"
+        rpy="0 0 0" />
+      <geometry>
+        <!-- <mesh
+          filename="package://hamr_description/meshes/base_link.stl" /> -->
+        <cylinder radius="0.225" length="0.1" />
       </geometry>
     </collision>
@@ -86,8 +87,9 @@
       <origin
         xyz="0 0 0"
-        rpy="0 1.5707963267949 0" />
-      <geometry>
-        <mesh
-          filename="package://hamr_description/meshes/right_wheel_link.stl" />
+        rpy="0 0 0" />
+      <geometry>
+        <!-- <mesh
+          filename="package://hamr_description/meshes/right_wheel_link.stl" /> -->
+        <cylinder radius="0.0762" length="0.0254" />
       </geometry>
     </collision>
@@ -138,6 +140,7 @@
         rpy="0 ${pi} 0" />
       <geometry>
-        <mesh
-          filename="package://hamr_description/meshes/left_wheel_link.stl" />
+        <!-- <mesh
+          filename="package://hamr_description/meshes/left_wheel_link.stl" /> -->
+        <cylinder radius="0.0762" length="0.0254" />
       </geometry>
     </collision>
@@ -238,6 +241,7 @@
         rpy="0 0 0" />
       <geometry>
-        <mesh
-          filename="package://hamr_description/meshes/right_caster_wheel_link.stl" />
+        <!-- <mesh
+          filename="package://hamr_description/meshes/right_caster_wheel_link.stl" /> -->
+        <cylinder radius="0.0508" length="0.0222" />
       </geometry>
     </collision>
@@ -288,6 +292,7 @@
         rpy="0 0 0" />
       <geometry>
-        <mesh
-          filename="package://hamr_description/meshes/left_caster_link.stl" />
+        <!-- <mesh
+          filename="package://hamr_description/meshes/left_caster_link.stl" /> -->
+        <cylinder radius="0.0508" length="0.0222" />
       </geometry>
     </collision>
@@ -338,6 +343,7 @@
         rpy="0 0 0" />
       <geometry>
-        <mesh
-          filename="package://hamr_description/meshes/left_caster_wheel_link.stl" />
+        <!-- <mesh
+          filename="package://hamr_description/meshes/left_caster_wheel_link.stl" /> -->
+        <cylinder radius="0.0508" length="0.0222" />
       </geometry>
     </collision>
@@ -388,6 +394,7 @@
         rpy="-3.14159265358979 0 0" />
       <geometry>
-        <mesh
-          filename="package://hamr_description/meshes/turret_link.stl" />
+        <!-- <mesh
+          filename="package://hamr_description/meshes/turret_link.stl" /> -->
+        <cylinder radius="0.225" length="0.05" />
       </geometry>
     </collision>
