Commit message: Improved heightmap in Gazebo. Now a smooth vs rocky map. Used Gimp for Gaussian Blur. Modified URDF (and added virtual weights for wheels and casters) to ensure proper friction between ground 2.5D plane and HAMR. Also removed unintentional colcon build inside hamr_bringup.

File: hamr_description/urdf/hamr.urdf.xacro (robot description, xacro)
@@ -2,5 +2,5 @@
 <robot name="hamr" xmlns:xacro="http://www.ros.org/wiki/xacro">
     <xacro:include filename="common_properties.xacro" />
-    <xacro:include filename="hamr_sw.xacro" />
+    <xacro:include filename="hamr_sw_v_simplified.xacro" />
     <xacro:include filename="hamr_gazebo.xacro" />
     <xacro:include filename="camera.xacro" />

File: hamr_description/urdf/hamr_gazebo.xacro (robot description, xacro)
@@ -10,18 +10,18 @@
     </gazebo>
     <gazebo reference="right_caster_link">
-        <mu1 value="0.2" />
-        <mu2 value="0.2" />
+        <mu1 value="0.9" />
+        <mu2 value="0.9" />
     </gazebo>
     <gazebo reference="left_caster_link">
-        <mu1 value="0.2" />
-        <mu2 value="0.2" />
+        <mu1 value="0.9" />
+        <mu2 value="0.9" />
     </gazebo>
     <gazebo reference="right_caster_wheel_link">
-        <mu1 value="0.8" />
-        <mu2 value="0.8" />
+        <mu1 value="1.0" />
+        <mu2 value="1.0" />
     </gazebo>
     <gazebo reference="left_caster_wheel_link">
-        <mu1 value="0.8" />
-        <mu2 value="0.8" />
+        <mu1 value="1.0" />
+        <mu2 value="1.0" />
     </gazebo>
     <gazebo reference="turret_link">
@@ -70,15 +70,12 @@
             <!-- world-fixed frame for odom -->
             <odom_frame>odom</odom_frame>
-            <!-- body-fixed frame on your robot -->
             <robot_base_frame>base_footprint</robot_base_frame>
-            <!-- publish rate (Hz) -->
             <odom_publish_frequency>50</odom_publish_frequency>
             <!-- ROS2 topics -->
             <odom_topic>/model/hamr/odometry</odom_topic>
-            <!-- publish the TF on the standard /tf topic -->
             <tf_topic>/model/hamr/tf</tf_topic>
             <!-- 2D odometry -->
             <dimensions>2</dimensions>
-            <!-- <xyz_offset>0.284843388017437 0.203598611982565 0</xyz_offset> -->
+            <!-- <xyz_offset>0.284843388017437 0.203598611982565 0</xyz_offset> didnt work well - rviz bugs -->
         </plugin>
     </gazebo>

File: hamr_description/urdf/hamr_sw_simplified.xacro (robot description, xacro)
@@ -46,9 +46,10 @@
     <collision>
       <origin
-        xyz="0 0 0"
-        rpy="0 0 0" />
-      <geometry>
-        <mesh
-          filename="package://hamr_description/meshes/base_link.stl" />
+        xyz="0.198549611345678 -0.271316507443243 0.0289830936800706"
+        rpy="0 0 0" />
+      <geometry>
+        <!-- <mesh
+          filename="package://hamr_description/meshes/base_link.stl" /> -->
+        <cylinder radius="0.225" length="0.1" />
       </geometry>
     </collision>
@@ -238,6 +239,7 @@
         rpy="0 0 0" />
       <geometry>
-        <mesh
-          filename="package://hamr_description/meshes/right_caster_wheel_link.stl" />
+        <!-- <mesh
+          filename="package://hamr_description/meshes/right_caster_wheel_link.stl" /> -->
+        <cylinder radius="0.0508" length="0.0222" />
       </geometry>
     </collision>
@@ -288,6 +290,7 @@
         rpy="0 0 0" />
       <geometry>
-        <mesh
-          filename="package://hamr_description/meshes/left_caster_link.stl" />
+        <!-- <mesh
+          filename="package://hamr_description/meshes/left_caster_link.stl" /> -->
+        <cylinder radius="0.0508" length="0.0222" />
       </geometry>
     </collision>
@@ -338,6 +341,7 @@
         rpy="0 0 0" />
       <geometry>
-        <mesh
-          filename="package://hamr_description/meshes/left_caster_wheel_link.stl" />
+        <!-- <mesh
+          filename="package://hamr_description/meshes/left_caster_wheel_link.stl" /> -->
+        <cylinder radius="0.0508" length="0.0222" />
       </geometry>
     </collision>
@@ -388,6 +392,7 @@
         rpy="-3.14159265358979 0 0" />
       <geometry>
-        <mesh
-          filename="package://hamr_description/meshes/turret_link.stl" />
+        <!-- <mesh
+          filename="package://hamr_description/meshes/turret_link.stl" /> -->
+        <cylinder radius="0.225" length="0.05" />
       </geometry>
     </collision>

File: hamr_description/urdf/hamr_sw_v_simplified.xacro (robot description, xacro)
@@ -46,9 +46,10 @@
     <collision>
       <origin
-        xyz="0 0 0"
-        rpy="0 0 0" />
-      <geometry>
-        <mesh
-          filename="package://hamr_description/meshes/base_link.stl" />
+        xyz="0.198549611345678 -0.271316507443243 0.0289830936800706"
+        rpy="0 0 0" />
+      <geometry>
+        <!-- <mesh
+          filename="package://hamr_description/meshes/base_link.stl" /> -->
+        <cylinder radius="0.225" length="0.1" />
       </geometry>
     </collision>
@@ -60,5 +61,5 @@
         rpy="0 1.5707963267949 0" />
       <mass
-        value="0.201354791790072" />
+        value="${20 * 0.201354791790072}" />
       <inertia
         ixx="0.000633771005763446"
@@ -86,8 +87,9 @@
       <origin
         xyz="0 0 0"
-        rpy="0 1.5707963267949 0" />
-      <geometry>
-        <mesh
-          filename="package://hamr_description/meshes/right_wheel_link.stl" />
+        rpy="0 0 0" />
+      <geometry>
+        <!-- <mesh
+          filename="package://hamr_description/meshes/right_wheel_link.stl" /> -->
+        <cylinder radius="0.0762" length="0.0254" />
       </geometry>
     </collision>
@@ -110,5 +112,5 @@
         rpy="0 ${pi} 0" />
       <mass
-        value="0.201354790396108" />
+        value="${20 * 0.201354790396108}" />
       <inertia
         ixx="0.000327993572579979"
@@ -135,9 +137,10 @@
     <collision>
       <origin
-        xyz="0 0 ${0.0254 / 2.0}"
+        xyz="0 0 0"
         rpy="0 ${pi} 0" />
       <geometry>
-        <mesh
-          filename="package://hamr_description/meshes/left_wheel_link.stl" />
+        <!-- <mesh
+          filename="package://hamr_description/meshes/left_wheel_link.stl" /> -->
+        <cylinder radius="0.0762" length="0.0254" />
       </geometry>
     </collision>
@@ -185,9 +188,10 @@
     <collision>
       <origin
-        xyz="0 0 0"
-        rpy="0 0 0" />
-      <geometry>
-        <mesh
-          filename="package://hamr_description/meshes/right_caster_link.stl" />
+        xyz="0 -0.0349 0"
+        rpy="0 0 0" />
+      <geometry>
+        <!-- <mesh
+          filename="package://hamr_description/meshes/right_caster_link.stl" /> -->
+        <box size="0.0508 0.0698500000000003 0.0222" />
       </geometry>
     </collision>
@@ -210,5 +214,5 @@
         rpy="0 0 0" />
       <mass
-        value="0.16654404953881" />
+        value="${1 * 0.16654404953881}" />
       <inertia
         ixx="0.000108847088077107"
@@ -238,6 +242,7 @@
         rpy="0 0 0" />
       <geometry>
-        <mesh
-          filename="package://hamr_description/meshes/right_caster_wheel_link.stl" />
+        <!-- <mesh
+          filename="package://hamr_description/meshes/right_caster_wheel_link.stl" /> -->
+        <cylinder radius="0.0508" length="0.0222" />
       </geometry>
     </collision>
@@ -285,9 +290,10 @@
     <collision>
       <origin
-        xyz="0 0 0"
-        rpy="0 0 0" />
-      <geometry>
-        <mesh
-          filename="package://hamr_description/meshes/left_caster_link.stl" />
+        xyz="0 -0.0349 0"
+        rpy="0 0 0" />
+      <geometry>
+        <!-- <mesh
+          filename="package://hamr_description/meshes/left_caster_link.stl" /> -->
+        <box size="0.0508 0.0698500000000003 0.0222" />
       </geometry>
     </collision>
@@ -310,5 +316,5 @@
         rpy="0 0 0" />
       <mass
-        value="0.16654404953881" />
+        value="${1 * 0.16654404953881}" />
       <inertia
         ixx="0.000108847088077107"
@@ -338,6 +344,7 @@
         rpy="0 0 0" />
       <geometry>
-        <mesh
-          filename="package://hamr_description/meshes/left_caster_wheel_link.stl" />
+        <!-- <mesh
+          filename="package://hamr_description/meshes/left_caster_wheel_link.stl" /> -->
+        <cylinder radius="0.0508" length="0.0222" />
       </geometry>
     </collision>
@@ -388,6 +395,7 @@
         rpy="-3.14159265358979 0 0" />
       <geometry>
-        <mesh
-          filename="package://hamr_description/meshes/turret_link.stl" />
+        <!-- <mesh
+          filename="package://hamr_description/meshes/turret_link.stl" /> -->
+        <cylinder radius="0.225" length="0.05" />
       </geometry>
     </collision>
