Commit message: Added some visualization stuff in rviz and edited urdf a bit. tried implementing Gimbal controller but not complete yet, maybe a tf error - the roll jitters but pitch seems fine somehow. Next steps: improve URDF inertia and mass and also simplify collisions

File: compa_description/urdf/common_properties.urdf.xacro (robot description, xacro)
@@ -57,3 +57,12 @@
         </inertial>
     </xacro:macro>
+    <xacro:macro name="sphere_inertia" params="m r o_xyz o_rpy">
+        <inertial>
+            <mass value="${m}" />
+            <origin xyz="${o_xyz}" rpy="${o_rpy}" />
+            <inertia ixx="${(2/5) * m * r*r}" ixy="0" ixz="0"
+                    iyy="${(2/5) * m * r*r}" iyz="0"
+                    izz="${(2/5) * m * r*r}" />
+        </inertial>
+    </xacro:macro>
 </robot>

File: compa_description/urdf/compa.urdf.xacro (robot description, xacro)
@@ -6,4 +6,5 @@
   <!-- <xacro:include filename="camera.urdf.xacro" /> -->
   <xacro:include filename="compa_gazebo.urdf.xacro" />
+  <!-- Base -->
   <link name="base_footprint" />
   <joint name="base_joint" type="fixed">
@@ -51,4 +52,5 @@
     </collision>
   </link>
+  <!-- Left Rocker -->
   <link name="left_rocker_link">
     <inertial>
@@ -82,9 +84,10 @@
     <collision>
       <origin
-        xyz="0 0 0"
-        rpy="0 0 0" />
-      <geometry>
-        <mesh
-          filename="package://compa_description/meshes/left_rocker_link.STL" />
+        xyz="0 -0.072 -0.021"
+        rpy="0 0 0" />
+      <geometry>
+        <!-- <mesh
+          filename="package://compa_description/meshes/left_rocker_link.STL" /> -->
+        <box size="0.6 0.037 0.05"/>
       </geometry>
     </collision>
@@ -152,4 +155,29 @@
       xyz="0 1 0" />
   </joint>
+  <link name="left_caster_wheel_link">
+    <xacro:sphere_inertia m="0.5" r="0.087"
+                        o_xyz="0 0 0" o_rpy="0 0 0" />
+    <collision>
+      <origin
+        xyz="0 0 0"
+        rpy="${pi/2} 0 0" />
+      <geometry>
+        <cylinder radius="0.087" length="0.05" />
+      </geometry>
+    </collision>
+  </link>
+  <joint name="left_rocker_left_caster_wheel_joint"
+    type="continuous">
+    <origin
+      xyz="0.315 -0.10422 -0.1647"
+      rpy="3.1416 0 0" />
+    <parent
+      link="left_rocker_link" />
+    <child
+      link="left_caster_wheel_link" />
+    <axis
+      xyz="0 1 0" />
+  </joint>
+  <!-- Right Rocker -->
   <link name="right_rocker_link">
     <inertial>
@@ -183,9 +211,10 @@
     <collision>
       <origin
-        xyz="0 0 0"
-        rpy="0 0 0" />
-      <geometry>
-        <mesh
-          filename="package://compa_description/meshes/right_rocker_link.STL" />
+        xyz="0 0.072 -0.021"
+        rpy="0 0 0" />
+      <geometry>
+        <!-- <mesh
+          filename="package://compa_description/meshes/right_rocker_link.STL" /> -->
+        <box size="0.6 0.037 0.05"/>
       </geometry>
     </collision>
@@ -253,4 +282,29 @@
       xyz="0 1 0" />
   </joint>
+  <link name="right_caster_wheel_link">
+    <xacro:sphere_inertia m="0.5" r="0.087"
+                        o_xyz="0 0 0" o_rpy="0 0 0" />
+    <collision>
+      <origin
+        xyz="0 0 0"
+        rpy="${pi/2} 0 0" />
+      <geometry>
+        <cylinder radius="0.087" length="0.05" />
+      </geometry>
+    </collision>
+  </link>
+  <joint name="right_rocker_right_caster_wheel_joint"
+    type="continuous">
+    <origin
+      xyz="0.315 0.10422 -0.1647"
+      rpy="3.1416 0 0" />
+    <parent
+      link="right_rocker_link" />
+    <child
+      link="right_caster_wheel_link" />
+    <axis
+      xyz="0 1 0" />
+  </joint>
+  <!-- Gimbal -->
   <link name="roll_link">
     <inertial>
@@ -406,4 +460,5 @@
       xyz="0 0 -1" />
   </joint>
+  <!-- ROCKER LINKS -->
   <link name="leverage_link">
     <inertial>
@@ -445,7 +500,6 @@
     </collision>
   </link>
-  <!-- BOGIE LINKS -->
   <joint name="base_leverage_joint"
-    type="continuous">
+    type="revolute">
     <origin
       xyz="0.2332 0 0.03826"
@@ -457,6 +511,7 @@
     <axis
       xyz="-1 0 0" />
-  </joint>
-  <!-- Right Side Bogie -->
+    <limit effort="20" velocity="1.0" lower="${-pi/12}" upper="${pi/12}"/>
+  </joint>
+  <!-- Right Side Rocker -->
   <link name="right_rod_sphere1_link">
     <inertial>
@@ -607,5 +662,5 @@
       link="right_rod_sphere2_link" />
   </joint>
-  <!-- Left Side Bogie -->
+  <!-- Left Side Rocker -->
   <link name="left_rod_sphere1_link">
     <inertial>
