Commit message: Getting closer to desired behavior. The error lies in the transform defintions in the urdf. Still some issues to fix in urdf and then controller to get: wheels in the front (right now in back), yaw turret is not right, and a lot of frames (gimbal etc) are wrongly defined

File: compa_description/urdf/compa.urdf.xacro (robot description, xacro)
@@ -4,10 +4,11 @@
   <!-- To import ball joint, camera and more -->
   <xacro:include filename="common_properties.urdf.xacro" />
-  <xacro:include filename="camera.urdf.xacro" />
+  <!-- <xacro:include filename="camera.urdf.xacro" /> -->
+  <xacro:include filename="compa_gazebo.urdf.xacro" />
   <link name="base_footprint" />
   <joint name="base_joint" type="fixed">
       <parent link="base_footprint" />
       <child link="base_link" />
-      <origin xyz="0 0 0.25042" rpy="0 0 0"/>
+      <origin xyz="0 0 0.25042" rpy="0 0 ${-pi/2}"/>
   </joint>
   <link name="base_link">
@@ -107,5 +108,5 @@
         rpy="0 0 0" />
       <mass
-        value="2.74378098590227" />
+        value="20.74378098590227" />
       <inertia
         ixx="0.00876644391195367"
@@ -208,5 +209,5 @@
         rpy="0 0 0" />
       <mass
-        value="2.74378098590227" />
+        value="20.74378098590227" />
       <inertia
         ixx="0.00876644391195365"
@@ -233,5 +234,5 @@
     <collision>
       <origin
-        xyz="0 0 ${pi}"
+        xyz="0 0 0"
         rpy="${pi/2} 0 0" />
       <geometry>

Commit message: Fixed the robot description. A bit confused by the behavoir of the robot (it insists to keep wheels at the back even with b negative. And when b is positive it breaks, but that makes sense since robot frame is set up for a negative b with drive wheels in the front

File: compa_description/urdf/compa.urdf.xacro (robot description, xacro)
@@ -10,5 +10,5 @@
       <parent link="base_footprint" />
       <child link="base_link" />
-      <origin xyz="0 0 0.25042" rpy="0 0 ${-pi/2}"/>
+      <origin xyz="0 0 0.25042" rpy="0 0 0"/>
   </joint>
   <link name="base_link">
@@ -30,5 +30,5 @@
       <origin
         xyz="0 0 0"
-        rpy="0 0 0" />
+        rpy="0 0 ${-pi/2}" />
       <geometry>
         <mesh
@@ -44,5 +44,5 @@
       <origin
         xyz="0 0 0"
-        rpy="0 0 0" />
+        rpy="0 0 ${-pi/2}" />
       <geometry>
         <mesh
@@ -93,6 +93,6 @@
     type="continuous">
     <origin
-      xyz="-0.184999999999999 0 0.0360999999999991"
-      rpy="0 0 -1.5707963267949" />
+      xyz="0 0.184999999999999 0.0360999999999991"
+      rpy="0 0 ${-pi}" />
     <parent
       link="base_link" />
@@ -194,6 +194,6 @@
     type="continuous">
     <origin
-      xyz="0.185 0 0.0361"
-      rpy="0 0 -1.5708" />
+      xyz="0 -0.185 0.0361"
+      rpy="0 0 ${-pi}" />
     <parent
       link="base_link" />
@@ -296,5 +296,5 @@
     <origin
       xyz="0 0 0.03826"
-      rpy="${-pi} 0 -1.5708" />
+      rpy="${-pi} 0 0" />
     <parent
       link="base_link" />
@@ -347,5 +347,5 @@
     <origin
       xyz="0.0035 0 0"
-      rpy="3.1416 0 0" />
+      rpy="3.1416 0 ${pi}" />
     <parent
       link="roll_link" />
@@ -373,5 +373,5 @@
       <origin
         xyz="0 0 0"
-        rpy="0 0 ${pi}" />
+        rpy="${pi} 0 ${pi}" />
       <geometry>
         <mesh
@@ -387,5 +387,5 @@
       <origin
         xyz="0 0 0"
-        rpy="0 0 ${pi}" />
+        rpy="${pi} 0 ${pi}" />
       <geometry>
         <mesh
@@ -398,5 +398,5 @@
     <origin
       xyz="0 0 0.0375"
-      rpy="0 0 ${pi}" />
+      rpy="${pi} 0 ${pi}" />
     <parent
       link="pitch_link" />
@@ -449,6 +449,6 @@
     type="continuous">
     <origin
-      xyz="0 0.2332 0.03826"
-      rpy="0 0 -1.5708" />
+      xyz="0.2332 0 0.03826"
+      rpy="0 0 ${-pi}" />
     <parent
       link="base_link" />

Commit message: Significantly improved compa simulation by simplifying COMPA Collisions and adding much finer resolution in the heightmap (actually makes a huge difference in how the robot sinks now). COMPA is able to go through very off road terrain in simulation now.

File: compa_description/urdf/compa.urdf.xacro (robot description, xacro)
@@ -14,18 +14,6 @@
   </joint>
   <link name="base_link">
-    <inertial>
-      <origin
-        xyz="-0.000339817170498122 0.00424231004595931 0.00197670802942906"
-        rpy="0 0 0" />
-      <mass
-        value="4.7675691308253" />
-      <inertia
-        ixx="0.139176668892902"
-        ixy="3.73786456449896E-05"
-        ixz="0.000406943794666223"
-        iyy="0.260635271329177"
-        iyz="-0.000613703988621289"
-        izz="0.12399220264823" />
-    </inertial>
+    <xacro:box_inertia m="4.77" x="0.45" y="0.45" z="0.05"
+                    o_xyz="0 0 0" o_rpy="0 0 ${-pi/2}" />
     <visual>
       <origin
@@ -47,6 +35,7 @@
         rpy="0 0 ${-pi/2}" />
       <geometry>
-        <mesh
-          filename="package://compa_description/meshes/base_link.STL" />
+        <!-- <mesh
+          filename="package://compa_description/meshes/base_link.STL" /> -->
+        <box size="0.45 0.45 0.05"/>
       </geometry>
     </collision>
@@ -318,18 +307,6 @@
   <!-- Gimbal -->
   <link name="roll_link">
-    <inertial>
-      <origin
-        xyz="0.00350000004402022 -5.16314840708076E-10 -4.00015491542477E-06"
-        rpy="0 0 0" />
-      <mass
-        value="0.944517139921142" />
-      <inertia
-        ixx="0.0181589556415456"
-        ixy="-6.29046022348623E-07"
-        ixz="-2.07968206915504E-11"
-        iyy="0.0184849903072778"
-        iyz="-7.02129324325875E-16"
-        izz="0.0364005003554526" />
-    </inertial>
+    <xacro:box_inertia m="0.944517139921142" x="0.35" y="0.35" z="0.05"
+                    o_xyz="0 0 0" o_rpy="0 0 0" />
     <visual>
       <origin
@@ -351,6 +328,7 @@
         rpy="0 0 0" />
       <geometry>
-        <mesh
-          filename="package://compa_description/meshes/roll_link.STL" />
+        <!-- <mesh
+          filename="package://compa_description/meshes/roll_link.STL" /> -->
+        <box size="0.35 0.35 0.05"/>
       </geometry>
     </collision>
@@ -402,6 +380,7 @@
         rpy="0 0 0" />
       <geometry>
-        <mesh
-          filename="package://compa_description/meshes/pitch_link.STL" />
+        <!-- <mesh
+          filename="package://compa_description/meshes/pitch_link.STL" /> -->
+        <box size="0.07 0.3 0.05"/>
       </geometry>
     </collision>
@@ -450,9 +429,10 @@
     <collision>
       <origin
-        xyz="0 0 0"
+        xyz="0 0 -0.127371508973676"
         rpy="${pi} 0 ${pi}" />
       <geometry>
-        <mesh
-          filename="package://compa_description/meshes/yaw_plate_link.STL" />
+        <!-- <mesh
+          filename="package://compa_description/meshes/yaw_plate_link.STL" /> -->
+        <cylinder radius="0.4" length="0.01"/>
       </geometry>
     </collision>
@@ -531,6 +511,7 @@
         rpy="0 0 0" />
       <geometry>
-        <mesh
-          filename="package://compa_description/meshes/leverage_link.STL" />
+        <!-- <mesh
+          filename="package://compa_description/meshes/leverage_link.STL" /> -->
+        <box size="0.01 0.45 0.07"/>
       </geometry>
     </collision>
@@ -584,6 +565,7 @@
         rpy="0 0 0" />
       <geometry>
-        <mesh
-          filename="package://compa_description/meshes/sphere_link.STL" />
+        <!-- <mesh
+          filename="package://compa_description/meshes/sphere_link.STL" /> -->
+        <sphere radius="0.0055"/>
       </geometry>
     </collision>
@@ -633,6 +615,7 @@
         rpy="0 0 ${pi/2}" />
       <geometry>
-        <mesh
-          filename="package://compa_description/meshes/rod_link.STL" />
+        <!-- <mesh
+          filename="package://compa_description/meshes/rod_link.STL" /> -->
+        <cylinder radius="0.0035" length="${2*0.07056 - 0.007}"/>
       </geometry>
     </collision>
@@ -683,6 +666,7 @@
         rpy="0 0 0" />
       <geometry>
-        <mesh
-          filename="package://compa_description/meshes/sphere_link.STL" />
+        <!-- <mesh
+          filename="package://compa_description/meshes/sphere_link.STL" /> -->
+        <sphere radius="0.0055"/>
       </geometry>
     </collision>
@@ -733,6 +717,7 @@
         rpy="0 0 0" />
       <geometry>
-        <mesh
-          filename="package://compa_description/meshes/sphere_link.STL" />
+        <!-- <mesh
+          filename="package://compa_description/meshes/sphere_link.STL" /> -->
+        <sphere radius="0.0055"/>
       </geometry>
     </collision>
@@ -782,6 +767,7 @@
         rpy="0 0 ${pi/2}" />
       <geometry>
-        <mesh
-          filename="package://compa_description/meshes/rod_link.STL" />
+        <!-- <mesh
+          filename="package://compa_description/meshes/rod_link.STL" /> -->
+        <cylinder radius="0.0035" length="${2*0.07056 - 0.007}"/>
       </geometry>
     </collision>
@@ -832,6 +818,7 @@
         rpy="0 0 0" />
       <geometry>
-        <mesh
-          filename="package://compa_description/meshes/sphere_link.STL" />
+        <!-- <mesh
+          filename="package://compa_description/meshes/sphere_link.STL" /> -->
+        <sphere radius="0.0055"/>
       </geometry>
     </collision>
