Commit message: Implemented Compa back wheel drive URDF (Front wheel drive requires updates if still needed). Added reference trajectory and orientation graphing in rviz. Properly implemented gimbal control (could be better tuned). Created a more intense and larger map using 2049x2049 res. Changed compa odom graph to show gimbal orientation (a bit broken, needs fix).

File: compa_description/urdf/compa_back.urdf.xacro (robot description, xacro)
@@ -11,25 +11,13 @@
       <parent link="base_footprint" />
       <child link="base_link" />
-      <origin xyz="0 0 0.25042" rpy="0 0 ${pi}"/>
+      <origin xyz="0 0 0.22" rpy="0 0 0"/>
   </joint>
   <link name="base_link">
-    <inertial>
-      <origin
-        xyz="-0.000339817170498122 0.00424231004595931 0.00197670802942906"
-        rpy="${-pi/2} 0 0" />
-      <mass
-        value="4.7675691308253" />
-      <inertia
-        ixx="0.139176668892902"
-        ixy="3.73786456449896E-05"
-        ixz="0.000406943794666223"
-        iyy="0.260635271329177"
-        iyz="-0.000613703988621289"
-        izz="0.12399220264823" />
-    </inertial>
-    <visual>
-      <origin
-        xyz="0 0 0"
-        rpy="0 0 ${-pi/2}" />
+    <xacro:box_inertia m="4.77" x="0.45" y="0.45" z="0.05"
+                    o_xyz="0 0 0" o_rpy="0 0 ${pi/2}" />
+    <visual>
+      <origin
+        xyz="0 0 0"
+        rpy="0 0 ${pi/2}" />
       <geometry>
         <mesh
@@ -45,13 +33,14 @@
       <origin
         xyz="0 0 0"
-        rpy="0 0 ${-pi/2}" />
-      <geometry>
-        <mesh
-          filename="package://compa_description/meshes/base_link.STL" />
+        rpy="0 0 ${pi/2}" />
+      <geometry>
+        <!-- <mesh
+          filename="package://compa_description/meshes/base_link.STL" /> -->
+        <box size="0.45 0.45 0.05"/>
       </geometry>
     </collision>
   </link>
   <!-- Left Rocker -->
-  <link name="left_rocker_link">
+  <link name="right_rocker_link">
     <!-- <inertial>
       <origin
@@ -76,5 +65,5 @@
       <geometry>
         <mesh
-          filename="package://compa_description/meshes/left_rocker_link.STL" />
+          filename="package://compa_description/meshes/f_right_rocker_link.STL" />
       </geometry>
       <material
@@ -90,22 +79,22 @@
       <geometry>
         <!-- <mesh
-          filename="package://compa_description/meshes/left_rocker_link.STL" /> -->
+          filename="package://compa_description/meshes/right_rocker_link.STL" /> -->
         <box size="0.6 0.037 0.05"/>
       </geometry>
     </collision>
   </link>
-  <joint name="base_left_rocker_joint"
+  <joint name="base_right_rocker_joint"
     type="continuous">
     <origin
-      xyz="0 0.184999999999999 0.0360999999999991"
-      rpy="0 0 ${-pi}" />
+      xyz="0 -0.184999999999999 0.0360999999999991"
+      rpy="0 0 0" />
     <parent
       link="base_link" />
     <child
-      link="left_rocker_link" />
+      link="right_rocker_link" />
     <axis
       xyz="0 1 0" />
   </joint>
-  <link name="left_wheel_link">
+  <link name="right_wheel_link">
     <!-- <inertial>
       <origin
@@ -127,9 +116,9 @@
     <visual>
       <origin
-        xyz="-0.001 -0.098 0"
-        rpy="0 0 0" />
-      <geometry>
-        <mesh
-          filename="package://compa_description/meshes/left_wheel_link.STL" />
+        xyz="0.001 0.098 0"
+        rpy="0 0 ${pi}" />
+      <geometry>
+        <mesh
+          filename="package://compa_description/meshes/f_right_wheel_link.STL" />
       </geometry>
       <material
@@ -148,5 +137,5 @@
     </collision>
   </link>
-  <joint name="left_rocker_left_wheel_joint"
+  <joint name="right_rocker_right_wheel_joint"
     type="continuous">
     <origin
@@ -154,11 +143,11 @@
       rpy="0 0 0" />
     <parent
-      link="left_rocker_link" />
-    <child
-      link="left_wheel_link" />
+      link="right_rocker_link" />
+    <child
+      link="right_wheel_link" />
     <axis
       xyz="0 1 0" />
   </joint>
-  <link name="left_caster_wheel_link">
+  <link name="right_caster_wheel_link">
     <xacro:cylinder_inertia m="5.0" r="0.087" h="0.05"
                         o_xyz="0 0 0" o_rpy="${pi/2} 0 0" />
@@ -172,5 +161,5 @@
     </collision>
   </link>
-  <joint name="left_rocker_left_caster_wheel_joint"
+  <joint name="right_rocker_right_caster_wheel_joint"
     type="continuous">
     <origin
@@ -178,12 +167,12 @@
       rpy="3.1416 0 0" />
     <parent
-      link="left_rocker_link" />
-    <child
-      link="left_caster_wheel_link" />
+      link="right_rocker_link" />
+    <child
+      link="right_caster_wheel_link" />
     <axis
       xyz="0 1 0" />
   </joint>
   <!-- Right Rocker -->
-  <link name="right_rocker_link">
+  <link name="left_rocker_link">
     <!-- <inertial>
       <origin
@@ -208,5 +197,5 @@
       <geometry>
         <mesh
-          filename="package://compa_description/meshes/right_rocker_link.STL" />
+          filename="package://compa_description/meshes/f_left_rocker_link.STL" />
       </geometry>
       <material
@@ -222,22 +211,22 @@
       <geometry>
         <!-- <mesh
-          filename="package://compa_description/meshes/right_rocker_link.STL" /> -->
+          filename="package://compa_description/meshes/left_rocker_link.STL" /> -->
         <box size="0.6 0.037 0.05"/>
       </geometry>
     </collision>
   </link>
-  <joint name="base_right_rocker_joint"
+  <joint name="base_left_rocker_joint"
     type="continuous">
     <origin
-      xyz="0 -0.185 0.0361"
-      rpy="0 0 ${-pi}" />
+      xyz="0 0.185 0.0361"
+      rpy="0 0 0" />
     <parent
       link="base_link" />
     <child
-      link="right_rocker_link" />
+      link="left_rocker_link" />
     <axis
       xyz="0 1 0" />
   </joint>
-  <link name="right_wheel_link">
+  <link name="left_wheel_link">
     <!-- <inertial>
       <origin
@@ -259,9 +248,9 @@
     <visual>
       <origin
-        xyz="-0.001 0.098 0"
-        rpy="0 0 0" />
-      <geometry>
-        <mesh
-          filename="package://compa_description/meshes/right_wheel_link.STL" />
+        xyz="-0.001 -0.098 0"
+        rpy="0 0 0" />
+      <geometry>
+        <mesh
+          filename="package://compa_description/meshes/f_left_wheel_link.STL" />
       </geometry>
       <material
@@ -280,5 +269,5 @@
     </collision>
   </link>
-  <joint name="right_rocker_right_wheel_joint"
+  <joint name="left_rocker_left_wheel_joint"
     type="continuous">
     <origin
@@ -286,11 +275,11 @@
       rpy="0 0 0" />
     <parent
-      link="right_rocker_link" />
-    <child
-      link="right_wheel_link" />
+      link="left_rocker_link" />
+    <child
+      link="left_wheel_link" />
     <axis
       xyz="0 1 0" />
   </joint>
-  <link name="right_caster_wheel_link">
+  <link name="left_caster_wheel_link">
     <xacro:cylinder_inertia m="5.0" r="0.087" h="0.05"
                         o_xyz="0 0 0" o_rpy="${pi/2} 0 0" />
@@ -304,5 +293,5 @@
     </collision>
   </link>
-  <joint name="right_rocker_right_caster_wheel_joint"
+  <joint name="left_rocker_left_caster_wheel_joint"
     type="continuous">
     <origin
@@ -310,7 +299,7 @@
       rpy="3.1416 0 0" />
     <parent
-      link="right_rocker_link" />
-    <child
-      link="right_caster_wheel_link" />
+      link="left_rocker_link" />
+    <child
+      link="left_caster_wheel_link" />
     <axis
       xyz="0 1 0" />
@@ -318,18 +307,6 @@
   <!-- Gimbal -->
   <link name="roll_link">
-    <inertial>
-      <origin
-        xyz="0.00350000004402022 -5.16314840708076E-10 -4.00015491542477E-06"
-        rpy="0 0 0" />
-      <mass
-        value="0.944517139921142" />
-      <inertia
-        ixx="0.0181589556415456"
-        ixy="-6.29046022348623E-07"
-        ixz="-2.07968206915504E-11"
-        iyy="0.0184849903072778"
-        iyz="-7.02129324325875E-16"
-        izz="0.0364005003554526" />
-    </inertial>
+    <xacro:box_inertia m="0.944517139921142" x="0.35" y="0.35" z="0.05"
+                    o_xyz="0 0 0" o_rpy="0 0 0" />
     <visual>
       <origin
@@ -351,6 +328,7 @@
         rpy="0 0 0" />
       <geometry>
-        <mesh
-          filename="package://compa_description/meshes/roll_link.STL" />
+        <!-- <mesh
+          filename="package://compa_description/meshes/roll_link.STL" /> -->
+        <box size="0.35 0.35 0.05"/>
       </geometry>
     </collision>
@@ -360,5 +338,5 @@
     <origin
       xyz="0 0 0.03826"
-      rpy="${-pi} 0 0" />
+      rpy="0 0 0" />
     <parent
       link="base_link" />
@@ -366,5 +344,5 @@
       link="roll_link" />
     <axis
-      xyz="-1 0 0" />
+      xyz="1 0 0" />
   </joint>
   <link name="pitch_link">
@@ -402,6 +380,7 @@
         rpy="0 0 0" />
       <geometry>
-        <mesh
-          filename="package://compa_description/meshes/pitch_link.STL" />
+        <!-- <mesh
+          filename="package://compa_description/meshes/pitch_link.STL" /> -->
+        <box size="0.07 0.3 0.05"/>
       </geometry>
     </collision>
@@ -410,6 +389,6 @@
     type="continuous">
     <origin
-      xyz="0.0035 0 0"
-      rpy="3.1416 0 ${pi}" />
+      xyz="-0.0035 0 0"
+      rpy="0 0 0" />
     <parent
       link="roll_link" />
@@ -451,8 +430,9 @@
       <origin
         xyz="0 0 0"
-        rpy="0 0 ${pi}" />
-      <geometry>
-        <mesh
-          filename="package://compa_description/meshes/yaw_plate_link.STL" />
+        rpy="0 0 0" />
+      <geometry>
+        <!-- <mesh
+          filename="package://compa_description/meshes/yaw_plate_link.STL" /> -->
+        <cylinder radius="0.4" length="0.01"/>
       </geometry>
     </collision>
@@ -468,5 +448,5 @@
       link="yaw_plate_link" />
     <axis
-      xyz="0 0 -1" />
+      xyz="0 0 1" />
   </joint>
   <!-- ROCKER LINKS -->
@@ -505,6 +485,7 @@
         rpy="0 0 0" />
       <geometry>
-        <mesh
-          filename="package://compa_description/meshes/leverage_link.STL" />
+        <!-- <mesh
+          filename="package://compa_description/meshes/leverage_link.STL" /> -->
+        <box size="0.01 0.45 0.07"/>
       </geometry>
     </collision>
@@ -513,6 +494,6 @@
     type="revolute">
     <origin
-      xyz="0.2332 0 0.03826"
-      rpy="0 0 ${-pi}" />
+      xyz="-0.2332 0 0.03826"
+      rpy="0 0 0" />
     <parent
       link="base_link" />
@@ -520,9 +501,9 @@
       link="leverage_link" />
     <axis
-      xyz="-1 0 0" />
+      xyz="1 0 0" />
     <limit effort="20" velocity="1.0" lower="${-pi/12}" upper="${pi/12}"/>
   </joint>
   <!-- Right Side Rocker -->
-  <link name="right_rod_sphere1_link">
+  <link name="left_rod_sphere1_link">
     <inertial>
       <origin
@@ -558,10 +539,11 @@
         rpy="0 0 0" />
       <geometry>
-        <mesh
-          filename="package://compa_description/meshes/sphere_link.STL" />
-      </geometry>
-    </collision>
-  </link>
-  <joint name="leverage_right_rod_sphere1_joint"
+        <!-- <mesh
+          filename="package://compa_description/meshes/sphere_link.STL" /> -->
+        <sphere radius="0.0055"/>
+      </geometry>
+    </collision>
+  </link>
+  <joint name="leverage_left_rod_sphere1_joint"
     type="fixed">
     <origin
@@ -571,7 +553,7 @@
       link="leverage_link" />
     <child
-      link="right_rod_sphere1_link" />
-  </joint>
-  <link name="right_rod_link">
+      link="left_rod_sphere1_link" />
+  </joint>
+  <link name="left_rod_link">
     <inertial>
       <origin
@@ -607,12 +589,13 @@
         rpy="0 0 ${pi/2}" />
       <geometry>
-        <mesh
-          filename="package://compa_description/meshes/rod_link.STL" />
-      </geometry>
-    </collision>
-  </link>
-  <xacro:ball_joint parent="right_rod_sphere1_link" child="right_rod_link"
-                   joint_prefix="right_rod_sphere1" roll_offset="-0.1075" pitch_offset="-0.0171" />
-  <link name="tmp_right_rod_sphere2_link">
+        <!-- <mesh
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