Commit message: Updated the urdf and preparing a more correct URDF for back wheel drive.

File: compa_description/urdf/camera.urdf.xacro (robot description, xacro)
@@ -10,5 +10,5 @@
             </geometry>
             <origin xyz="${camera_length / 2.0} 0 0" rpy="0 0 0" />
-            <material name="black" />
+            <!-- <material name="black" /> -->
         </visual>
         <collision>
@@ -25,5 +25,5 @@
         <parent link="yaw_plate_link" />
         <child link="camera_link" />
-        <origin xyz="0 0 0.1" rpy="0 0 ${-pi}"/>
+        <origin xyz="0 0 -0.15" rpy="0 0 ${-pi}"/>
     </joint>
     <!-- generate an optical frame

File: compa_description/urdf/common_properties.urdf.xacro (robot description, xacro)
@@ -38,8 +38,8 @@
             <limit lower="-${lim}" upper="${lim}" effort="1" velocity="1"/>
         </joint>
-        <joint name="${joint_prefix}_rev_z" type="revolute">
+        <joint name="${joint_prefix}_rev_z" type="continuous">
             <parent link="${joint_prefix}_t2"/><child link="${joint_prefix}_t3"/>
             <origin xyz="0 0 0" rpy="0 0 ${yaw_offset}"/><axis xyz="0 0 1"/>
-            <limit lower="-${lim}" upper="${lim}" effort="1" velocity="1"/>
+            <!-- <limit lower="-${lim}" upper="${lim}" effort="1" velocity="1"/> -->
         </joint>
         <joint name="${joint_prefix}_fixed" type="fixed">
@@ -66,3 +66,12 @@
         </inertial>
     </xacro:macro>
+    <xacro:macro name="cylinder_inertia" params="m r h o_xyz:='0 0 0' o_rpy:='0 0 0'">
+        <inertial>
+            <mass value="${m}" />
+            <origin xyz="${o_xyz}" rpy="${o_rpy}" />
+            <inertia ixx="${(m/12) * (3*r*r + h*h)}" ixy="0" ixz="0"
+                     iyy="${(m/12) * (3*r*r + h*h)}" iyz="0"
+                     izz="${(m/2) * (r*r)}" />
+        </inertial>
+    </xacro:macro>
 </robot>

File: compa_description/urdf/compa_back.urdf.xacro (robot description, xacro)
@@ -11,5 +11,5 @@
       <parent link="base_footprint" />
       <child link="base_link" />
-      <origin xyz="0 0 0.25042" rpy="0 0 0"/>
+      <origin xyz="0 0 0.25042" rpy="0 0 ${pi}"/>
   </joint>
   <link name="base_link">
@@ -17,5 +17,5 @@
       <origin
         xyz="-0.000339817170498122 0.00424231004595931 0.00197670802942906"
-        rpy="0 0 0" />
+        rpy="${-pi/2} 0 0" />
       <mass
         value="4.7675691308253" />
@@ -124,5 +124,5 @@
     <xacro:cylinder_inertia m="20.74378098590227" r="0.1075" h="0.083"
                         o_xyz="0 0 0"
-                        o_rpy="${pi/2} 0 0" />
+                        o_rpy="${-pi/2} 0 0" />
     <visual>
       <origin
@@ -142,5 +142,5 @@
       <origin
         xyz="0 0 0"
-        rpy="${pi/2} 0 0" />
+        rpy="${-pi/2} 0 0" />
       <geometry>
         <cylinder radius="0.1075" length="0.083" />
@@ -152,5 +152,5 @@
     <origin
       xyz="-0.27114 -0.14572 -0.1442"
-      rpy="3.1416 0 0" />
+      rpy="0 0 0" />
     <parent
       link="left_rocker_link" />
@@ -256,9 +256,9 @@
     <xacro:cylinder_inertia m="20.74378098590227" r="0.1075" h="0.083"
                         o_xyz="0 0 0"
-                        o_rpy="${pi/2} 0 0" />
+                        o_rpy="${-pi/2} 0 0" />
     <visual>
       <origin
         xyz="-0.001 0.098 0"
-        rpy="0 0 ${pi}" />
+        rpy="0 0 0" />
       <geometry>
         <mesh
@@ -274,5 +274,5 @@
       <origin
         xyz="0 0 0"
-        rpy="${pi/2} 0 0" />
+        rpy="${-pi/2} 0 0" />
       <geometry>
         <cylinder radius="0.1075" length="0.083" />
@@ -284,5 +284,5 @@
     <origin
       xyz="-0.27114 0.14572 -0.1442"
-      rpy="0 0 ${pi}" />
+      rpy="0 0 0" />
     <parent
       link="right_rocker_link" />
@@ -437,5 +437,5 @@
       <origin
         xyz="0 0 0"
-        rpy="${pi} 0 ${pi}" />
+        rpy="0 0 ${pi}" />
       <geometry>
         <mesh
@@ -451,5 +451,5 @@
       <origin
         xyz="0 0 0"
-        rpy="${pi} 0 ${pi}" />
+        rpy="0 0 ${pi}" />
       <geometry>
         <mesh
@@ -462,5 +462,5 @@
     <origin
       xyz="0 0 0.0375"
-      rpy="${pi} 0 ${pi}" />
+      rpy="0 0 0" />
     <parent
       link="pitch_link" />
@@ -469,30 +469,4 @@
     <axis
       xyz="0 0 -1" />
-  </joint>
-  <!-- Dummy link to visualize yaw axis -->
-  <link name="yaw_dummy_link">
-    <inertial>
-      <mass value="0.001"/>
-      <inertia ixx="1e-6" iyy="1e-6" izz="1e-6" ixy="0" ixz="0" iyz="0"/>
-    </inertial>
-    <visual name="yaw_dummy_visual">
-      <geometry>
-        <sphere radius="0.001"/>
-      </geometry>
-    </visual>
-    <collision name="yaw_dummy_collision">
-      <geometry>
-        <sphere radius="0.03"/>
-      </geometry>
-    </collision>
-  </link>
-  <joint name="yaw_plate_fixed_joint" type="revolute">
-    <origin xyz="0 0 0.075" rpy="${pi} 0 0"/>
-    <parent link="yaw_plate_link"/>
-    <child  link="yaw_dummy_link"/>
-    <axis xyz="0 0 1"/>
-    <!-- Lock at 0 lower=upper=0; add large effort + damping so it stays put -->
-    <limit lower="0" upper="0" effort="1e6" velocity="0"/>
-    <dynamics damping="100" friction="1.0"/>
   </joint>
   <!-- ROCKER LINKS -->

Commit message: Tuned the gimbal, fixed odom graphing and added a new node for it. Added camera for visualization - the gimbal does a pretty good job but it doesnt smooth out high frequency disturbances (which is expected) - we probably need a physical damper.

File: compa_description/urdf/camera.urdf.xacro (robot description, xacro)
@@ -25,5 +25,5 @@
         <parent link="yaw_plate_link" />
         <child link="camera_link" />
-        <origin xyz="0 0 -0.15" rpy="0 0 ${-pi}"/>
+        <origin xyz="0 0 0.25" rpy="0 0 0"/>
     </joint>
     <!-- generate an optical frame

File: compa_description/urdf/compa_back.urdf.xacro (robot description, xacro)
@@ -4,5 +4,5 @@
   <!-- To import ball joint, camera and more -->
   <xacro:include filename="common_properties.urdf.xacro" />
-  <!-- <xacro:include filename="camera.urdf.xacro" /> -->
+  <xacro:include filename="camera.urdf.xacro" />
   <xacro:include filename="compa_gazebo.urdf.xacro" />
   <!-- Base -->
